File: ESP32_sensor_board/esp32-c3-02.kicad_sch (KiCad schematic)
At the start: 30 parts, among them J3 GSD090012SEU, U3 ESP32-C3-WROOM-02-H4, U4 CP2102N-Axx-xQFN20, U5 USBLC6-2SC6, U6 W25Q32JVSSIQ

Commit message: Schematic design section 3 completed
Parts:
- C10, C11, C13, C14, C8: footprint (none) -> Capacitor_SMD:C_0805_2012Metric
- C12, C7, C9: footprint (none) -> footprints:T491A106K010AT
- J3: footprint GSD090012SEU:AMPHENOL_GSD090012SEU -> footprints:AMPHENOL_GSD090012SEU
- LED5: footprint LTST-C170KGKT:DIOC200X125X110 -> footprints:DIOC200X125X110
- LED6: footprint LTST-C170KRKT:DIOC200X125X110 -> footprints:DIOC200X125X110
- R11, R12, R13, R14, R15, R16, R18, R19, R20, R22: footprint (none) -> Resistor_SMD:R_0805_2012Metric
- TP1, TP2, TP3, TP4, TP5: footprint (none) -> TestPoint:TestPoint_Pad_D1.0mm
- U3: footprint ESP32-C3-WROOM-02-H4:MODULE_ESP32-C3-WROOM-02-H4 -> footprints:MODULE_ESP32-C3-WROOM-02-H4
- U4: footprint Package_DFN_QFN:SiliconLabs_QFN-20-1EP_3x3mm_P0.5mm -> footprints:WFQFN-20
- U6: footprint W25Q32JVSSIQ:SOIC127P790X216-8N -> footprints:SOIC127P790X216-8N
Connections:
- net DTS renamed DTR
Other:
- sheet Sensors ports: added MIC_OUT, PHOTO_C, SCL, SDA; removed none
- sheet User interface ports: added BOOT, DTR, EN, GPIO_18, GPIO_19, GPIO_8, RTS, SCL, SDA; removed none

Commit message: Layout design section 3 in progress
Connections:
- net CLK: now also TP3.1
- net SCLK: no longer TP3.1
Changed lines of the file:
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@@
 		)
 	)
-	(label "SCLK"
+	(label "CLK"
 		(at 140.97 137.16 0)
 		(effects

Commit message: Prototype 2 completed
Connections:
- net CS_SD: now also U3.4 (IO5); no longer U3.18 (IO0)
- net MIC_OUT: now also U3.18 (IO0); no longer U3.4 (IO5)
Changed lines of the file:
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@@
 		(title "ESP32 C3, USB and, flash memory")
 		(date "2025-06-02")
-		(rev "1")
+		(rev "2")
 		(company "Ing. Andrés Chaparro")
 	)
@@
 		)
 	)
-	(label "MIC_OUT"
-		(at 187.96 62.23 180)
-		(effects
-			(font
-				(size 1.27 1.27)
-			)
-			(justify right bottom)
-		)
-	)
 	(label "VBUS_DI"
 		(at 72.39 50.8 180)
@@
 		)
 	)
+	(label "MIC_OUT"
+		(at 187.96 49.53 180)
+		(effects
+			(font
+				(size 1.27 1.27)
+			)
+			(justify right bottom)
+		)
+	)
 	(label "MOSI_DI"
 		(at 140.97 121.92 0)
@@
 	)
 	(label "CS_SD"
-		(at 187.96 49.53 180)
-		(effects
-			(font
+		(at 187.96 62.23 180)
+		(effects
+			(font
