File: ESP32_sensor_board/user_inferface.kicad_sch (KiCad schematic)
At the start: 0 parts

Commit message: Schematic design section 2 completed
Other:
- title: ESP32 sensor board - Root -> (none)
Changed lines of the file:
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@@
 	(paper "A4")
 	(title_block
-		(title "ESP32 sensor board - Root")
 		(date "2025-06-02")
 		(rev "1")

Commit message: Schematic design section 3 completed
Parts:
- added C21: 0.1u, Capacitor_SMD:C_0805_2012Metric, symbol Device:C
- added C22: 1u, Capacitor_SMD:C_0805_2012Metric, symbol Device:C
- added J4: Conn_01x04_Pin, Connector_PinHeader_2.54mm:PinHeader_1x04_P2.54mm_Vertical, symbol Connector:Conn_01x04_Pin
- added J6: Conn_01x05_Pin, Connector_PinHeader_2.54mm:PinHeader_1x05_P2.54mm_Vertical, symbol Connector:Conn_01x05_Pin
- added Q2, Q3: BC817, Package_TO_SOT_SMD:SOT-23, symbol Transistor_BJT:BC817
- added R32, R33, R34: 10K, Resistor_SMD:R_0805_2012Metric, symbol Device:R
- added S1, S2: USLPT2819DT2TR, footprints:SW_USLPT2819DT2TR, symbol USLPT2819DT2TR:USLPT2819DT2TR
Connections:
- new net +3.3V: J4.1 (Pin_1), J6.1 (Pin_1), R32.1
- new net BOOT: C21.1, Q3.2 (E), S1.3, S1.4
- new net B_Q2: Q2.1 (B), R33.2
- new net B_Q3: Q3.1 (B), R34.2
- new net DTR: Q3.3 (C), R33.1
- new net EN: C22.1, Q2.3 (C), R32.2, S2.3, S2.4
- new net GND: C21.2, C22.2, J4.4 (Pin_4), J6.5 (Pin_5), S1.1, S1.2, S2.1, S2.2
- new net GPIO_18: J6.3 (Pin_3)
- new net GPIO_19: J6.4 (Pin_4)
- new net GPIO_8: J6.2 (Pin_2)
- new net RTS: Q2.2 (E), R34.1
- new net SCL: J4.3 (Pin_3)
- new net SDA: J4.2 (Pin_2)
Other:
- note added: "BOOT"
- note added: "Breakout for remaining pins"
- note added: "OLED display connector (I2C)"
- note added: "RESET"
- note added: "RESET and BOOT buttons"
- title: (none) -> User Interface

Commit message: Prototype 2 completed
Parts:
- removed S1, S2: USLPT2819DT2TR, footprints:SW_USLPT2819DT2TR, symbol USLPT2819DT2TR:USLPT2819DT2TR
- added S1, S2: TL3305AF260QG, footprints:SW_TL3305AF260QG, symbol TL3305AF260QG:TL3305AF260QG
Connections:
- net BOOT: now also Q3.3 (C), S1.1, S1.2; no longer Q3.2 (E)
- net DTR: now also Q3.2 (E); no longer Q3.3 (C)
- net EN: now also S2.1, S2.2
- net GND: now also S1.3, S1.4, S2.3, S2.4
Other:
- moved on the sheet: C21, C22, R32
